Commit message: add basic training and eval of ARS policy for pupper add joint limits to pupper_v2a.urdf

File: puppersim/data/pupper_v2a.urdf (robot description, URDF)
Before this commit: robot pupper_v2_dji, 17 links, 16 joints
Links:
- link leftFrontLeg: mass 0.50000 -> 0.20000
- link leftRearLeg: mass 0.50000 -> 0.20000
- link rightFrontLeg: mass 0.50000 -> 0.20000
- link rightRearLeg: mass 0.50000 -> 0.20000
Joints:
- joint leftFrontLegMotor: limit (none) -> lower=-0.2 upper=.2 effort=100 velocity=100; type continuous -> revolute
- joint leftFrontLowerLegMotor: limit (none) -> lower=-2.4 upper=-.5 effort=100 velocity=100; type continuous -> revolute
- joint leftFrontUpperLegMotor: limit (none) -> lower=0.0 upper=.8 effort=100 velocity=100; type continuous -> revolute
- joint leftRearLegMotor: limit (none) -> lower=-0.2 upper=.2 effort=100 velocity=100; type continuous -> revolute
- joint leftRearLowerLegMotor: limit (none) -> lower=-2.4 upper=-.5 effort=100 velocity=100; type continuous -> revolute
- joint leftRearUpperLegMotor: limit (none) -> lower=0.0 upper=.8 effort=100 velocity=100; type continuous -> revolute
- joint rightFrontLegMotor: limit (none) -> lower=-0.2 upper=.2 effort=100 velocity=100; type continuous -> revolute
- joint rightFrontLowerLegMotor: limit (none) -> lower=-2.4 upper=-.5 effort=100 velocity=100; type continuous -> revolute
- joint rightFrontUpperLegMotor: limit (none) -> lower=0.0 upper=.8 effort=100 velocity=100; type continuous -> revolute
- joint rightRearLegMotor: limit (none) -> lower=-0.2 upper=.2 effort=100 velocity=100; type continuous -> revolute
- joint rightRearLowerLegMotor: limit (none) -> lower=-2.4 upper=-.5 effort=100 velocity=100; type continuous -> revolute
- joint rightRearUpperLegMotor: limit (none) -> lower=0.0 upper=.8 effort=100 velocity=100; type continuous -> revolute

Commit message: remove visuals from pupper urdf, the meshes use up way too much memory, preventing training on Mac M1 (out of memory in Ray)

File: puppersim/data/pupper_v2a.urdf (robot description, URDF)
Before this commit: robot pupper_v2_dji, 17 links, 16 joints
Links:
- link leftFrontLeg: geometry collision cylinder length=0.075 radius=0.015
- link leftFrontLowerLeg: geometry collision box size=0.00951 0.012 0.10758
- link leftFrontToe: geometry collision sphere radius=0.0095
- link leftFrontUpperLeg: geometry collision cylinder length=0.065 radius=0.015
- link leftRearLeg: geometry collision cylinder length=0.075 radius=0.015
- link leftRearLowerLeg: geometry collision box size=0.00951 0.012 0.10758
- link leftRearToe: geometry collision sphere radius=0.0095
- link leftRearUpperLeg: geometry collision cylinder length=0.065 radius=0.015
- link pupper_v2_dji_chassis: geometry collision mesh filename=meshes/Cube.003.obj scale=1.0 1.0 1.0
- link rightFrontLeg: geometry collision cylinder length=0.075 radius=0.015
- link rightFrontLowerLeg: geometry collision box size=0.00953 0.012 0.10758
- link rightFrontToe: geometry collision sphere radius=0.0095
- link rightFrontUpperLeg: geometry collision cylinder length=0.065 radius=0.015
- link rightRearLeg: geometry collision cylinder length=0.075 radius=0.015
- link rightRearLowerLeg: geometry collision box size=0.00953 0.012 0.10758
- link rightRearToe: geometry collision sphere radius=0.0095
- link rightRearUpperLeg: geometry collision cylinder length=0.065 radius=0.015

Commit message: toes should be fixed, not floating

File: puppersim/data/pupper_v2a.urdf (robot description, URDF)
Before this commit: robot pupper_v2_dji, 17 links, 16 joints
Joints:
- joint leftFrontToe: type floating -> fixed
- joint leftRearToe: type floating -> fixed
- joint rightFrontToe: type floating -> fixed
- joint rightRearToe: type floating -> fixed
